File: stm32f103_ethernet_shield.sch (EAGLE design)
At the start: 6 parts

Commit message: Removed old backups
Connections:
- net 5V: now also POWER.CG1; no longer POWER.CTT, POWER.TD+
- net GND@3: now also POWER.CTT, POWER.S2; no longer POWER.CG1
- net RESET: now also POWER.TD+
